File: PCB/PCBv0.1/SolarGPS.sch (KiCad schematic (older format))
At the start: 72 parts, among them J1 Conn_01x10_Female, J2 USB_B_Micro, J4 Conn_02x05_Odd_Even, SW1 SW_Push, SW2 SW_Push, U1 BQ25570, U2 MAX-M8Q, U3 STM32L433CCUx, U4 MIC5225, U5 MAX40200AUK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

Commit message: Update Test bed to 2.7Vcc
Parts:
- ROUT1: value 5.23M -> 5.76M
- ROUT2: value 7.68M -> 7.32M
Other:
- note added: "VBATOV = 5.453\nVBATOK = 2.677\nVBATOKHYST = 2.971\nVOUT = 2.748"
- note removed: "VBATOV = 5.453\nVBATOK = 2.677\nVBATOKHYST = 2.971\nVOUT = 2.987"
Changed lines of the file:
@@
 P 1550 7100
 F 0 "ROUT2" V 1625 7100 50  0000 C CNN
-F 1 "7.68M" V 1475 7100 50  0000 C CNN
+F 1 "7.32M" V 1475 7100 50  0000 C CNN
 F 2 "Resistor_SMD:R_0603_1608Metric" H 1550 7100 50  0001 C CNN
 F 3 "~" H 1550 7100 50  0001 C CNN
@@
 P 1300 7100
 F 0 "ROUT1" V 1375 7100 50  0000 C CNN
-F 1 "5.23M" V 1225 7100 50  0000 C CNN
+F 1 "5.76M" V 1225 7100 50  0000 C CNN
 F 2 "Resistor_SMD:R_0603_1608Metric" H 1300 7100 50  0001 C CNN
 F 3 "~" H 1300 7100 50  0001 C CNN
@@
 Shunt
 Text Notes 1500 7875 0    50   ~ 0
-VBATOV      = 5.453\nVBATOK      = 2.677\nVBATOKHYST = 2.971\nVOUT        = 2.987
+VBATOV      = 5.453\nVBATOK      = 2.677\nVBATOKHYST = 2.971\nVOUT        = 2.748
 $Comp
 L Device:CP C16
