File: PCB/PCBv1.0/SolarGPS.kicad_pcb (KiCad board)
At the start: 2 copper layers, 73 x 27 mm, 57 parts, among them J1 Conn_01x10_Female, J2 Solar1+, J3 GND, J4 Conn_02x05_Odd_Even, J5 Solar2+, J6 GND, J7 Screw_Terminal_01x01, U2 MAX-M10Q, U3 MAX40200AUK, U4 STM32WB5MMGH6TR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

Commit message: Cost Reduction
Parts:
- removed C24: 1uF, Capacitor_SMD:C_0603_1608Metric
- removed U3: MAX40200AUK, Package_TO_SOT_SMD:SOT-23-5
- added C21: 1uF, Capacitor_SMD:C_0603_1608Metric, F.Cu at (109.3, 62.9)
Connections:
- U2 pad 6: VDD -> Net-(U2-Pad6)
- U2 pad 7: /GPSVCC -> VDD
- U2 pad 8: /GPSVCC -> VDD
- U4 pad 41: GPSEN -> Net-(U4-Pad41)
Routing:
- net GPSEN: track 59.1 -> 0.00 mm, vias 2 -> 0
- net /GPSVCC: track 10.8 -> 0.00 mm
- net VDD: track 145.4 -> 140.0 mm
- net SOLAR_SENSE1: track 61.2 -> 60.5 mm
Other:
- board text added: "GNSS"

Commit message: Most Cost Savings
Parts:
- removed C4: 1uF, Capacitor_SMD:C_0603_1608Metric
- removed R1: 1M, Resistor_SMD:R_0603_1608Metric
Connections:
- U7 pad 1: Net-(C4-Pad2) -> VBAT
Routing:
- net VBAT: track 75.1 -> 79.6 mm, vias 2 -> 3
- net Net-(C4-Pad2): track 4.16 -> 0.00 mm
- net GND: track 27.1 -> 31.0 mm, vias 108 -> 109
