File: PCB/PCBv1.0/SolarGPS.sch (KiCad schematic (older format))
At the start: 57 parts, among them J1 Conn_01x10_Female, J2 Solar1+, J3 GND, J4 Conn_02x05_Odd_Even, J5 Solar2+, J6 GND, J7 Screw_Terminal_01x01, U2 MAX-M10Q, U3 MAX40200AUK, U4 STM32WB5MMGH6TR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

Commit message: Cost Reduction
Parts:
- removed C24: 1uF, Capacitor_SMD:C_0603_1608Metric, symbol Device:C_Small
- removed U3: MAX40200AUK, Package_TO_SOT_SMD:SOT-23-5, symbol Analog_Switch:MAX40200AUK
- added C21: 1uF, Capacitor_SMD:C_0603_1608Metric, symbol Device:C_Small
Connections:
- net GPSVCC is gone; now on net VDD: U2.7 (VCC_IO), U2.8 (VCC)
- net GND: now also C21.2
- net VDD: now also C21.1; no longer U2.6 (V_BCKP)
- net GPSEN: no longer names the net of U4.41 (PB12)
- no-connect marks 24 -> 25

Commit message: Most Cost Savings
Parts:
- removed C4: 1uF, Capacitor_SMD:C_0603_1608Metric, symbol Device:C_Small
- removed R1: 1M, Resistor_SMD:R_0603_1608Metric, symbol Device:R_Small
Connections:
- net VBAT: now also U7.1 (EN)
Other:
- moved on the sheet: C12, C14, C15, C17, C19, C2, C5, C7, C8, L2, R4, R5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

Commit message: Tweak part numbers
Parts:
- D1, D3: Part B0530WS -> B0530WS-TP
- L2: Part DFE201612E -> CIGT201208EHR47MNE
- U2: value MAX-M10Q -> MAX-M10S
Changed lines of the file:
@@
 P 2275 2975
 F 0 "U2" H 2850 3550 50  0000 C CNN
-F 1 "MAX-M10Q" H 2975 3450 50  0000 C CNN
+F 1 "MAX-M10S" H 2975 3450 50  0000 C CNN
 F 2 "RF_GPS:ublox_MAX" H 2675 2325 50  0001 C CNN
 F 3 "https://www.u-blox.com/sites/default/files/MAX-M8-FW3_DataSheet_%28UBX-15031506%29.pdf" H 2275 2975 50  0001 C CNN
@@
 F 2 "Inductor_SMD:L_0806_2016Metric" H 4800 6400 50  0001 C CNN
 F 3 "~" H 4800 6400 50  0001 C CNN
-F 4 "DFE201612E" V 4800 6400 50  0001 C CNN "Part"
+F 4 "CIGT201208EHR47MNE" V 4800 6400 50  0001 C CNN "Part"
 	1    4800 6400
 	0    -1   -1   0
@@
 F 2 "Diode_SMD:D_SOD-323_HandSoldering" V 1725 4900 50  0001 C CNN
 F 3 "~" V 1725 4900 50  0001 C CNN
-F 4 "B0530WS" H 1725 4900 50  0001 C CNN "Part"
+F 4 "B0530WS-TP" H 1725 4900 50  0001 C CNN "Part"
 	1    1725 4900
 	1    0    0    1
@@
 F 2 "Diode_SMD:D_SOD-323_HandSoldering" V 1725 5425 50  0001 C CNN
 F 3 "~" V 1725 5425 50  0001 C CNN
-F 4 "B0530WS" H 1725 5425 50  0001 C CNN "Part"
+F 4 "B0530WS-TP" H 1725 5425 50  0001 C CNN "Part"
 	1    1725 5425
 	1    0    0    1

Commit message: Change VCC to 2.87 Remove LCD connector
Parts:
- R4: value 412k -> 432k
Other:
- note added: "VOUT = 2.87"
- note removed: "VOUT = 2.76"
Changed lines of the file:
@@
 P 5525 6900
 F 0 "R4" H 5675 6925 50  0000 C CNN
-F 1 "412k" H 5650 6850 50  0000 C CNN
+F 1 "432k" H 5650 6850 50  0000 C CNN
 F 2 "Resistor_SMD:R_0603_1608Metric" H 5525 6900 50  0001 C CNN
 F 3 "~" H 5525 6900 50  0001 C CNN
@@
 $EndComp
 Text Notes 5375 6600 0    50   ~ 0
-VOUT = 2.76
+VOUT = 2.87
 $Comp
 L Device:C_Small C2

Commit message: tweak PCB1.1 add some notes
Parts:
- J7: Part 7781 -> 7792
Changed lines of the file:
@@
 F 2 "Veridian-Library-KiCad:Right Angle Screw Terminal M3M4" H 7875 7175 50  0001 C CNN
 F 3 "~" H 7875 7175 50  0001 C CNN
-F 4 "7781" V 7875 7175 50  0001 C CNN "Part"
+F 4 "7792" V 7875 7175 50  0001 C CNN "Part"
 F 5 "Keystone Electronics" V 7875 7175 50  0001 C CNN "Manufacture"
 	1    7875 7175
