File: PCB/PCBv1.1/SolarGPS.kicad_sch (KiCad schematic)
At the start: 56 parts, among them J1 Conn_01x10_Female, J2 Solar1+, J3 GND, J4 Conn_02x03_Odd_Even, J5 Solar2+, J6 GND, J7 Screw_Terminal_01x01, U1 STM32L011G3Ux, U2 MAX-M10Q, U5 BQ25505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

Commit message: Revise
Parts:
- C14, C17: value 10F -> 15F; footprint Veridian-Library-KiCad:SCCT20E106SRB -> Heliograph:SCCT30E156SRB; Part SCCT20E106SRB -> SCCT30E156SRB
Changed lines of the file:
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@@
       (effects (font (size 1.27 1.27)) (justify left))
     )
-    (property "Value" "10F" (id 1) (at 95.0722 170.688 0)
-      (effects (font (size 1.27 1.27)) (justify left))
-    )
-    (property "Footprint" "Veridian-Library-KiCad:SCCT20E106SRB" (id 2) (at 93.0402 173.355 0)
+    (property "Value" "15F" (id 1) (at 95.0722 170.688 0)
+      (effects (font (size 1.27 1.27)) (justify left))
+    )
+    (property "Footprint" "Heliograph:SCCT30E156SRB" (id 2) (at 93.0402 173.355 0)
       (effects (font (size 1.27 1.27)) hide)
     )
@@
       (effects (font (size 1.27 1.27)) hide)
     )
-    (property "Part" "SCCT20E106SRB" (id 4) (at 92.075 169.545 0)
+    (property "Part" "SCCT30E156SRB" (id 4) (at 92.075 169.545 0)
       (effects (font (size 1.27 1.27)) hide)
     )
@@
       (effects (font (size 1.27 1.27)) (justify left))
     )
-    (property "Value" "10F" (id 1) (at 95.0722 178.308 0)
-      (effects (font (size 1.27 1.27)) (justify left))
-    )
-    (property "Footprint" "Veridian-Library-KiCad:SCCT20E106SRB" (id 2) (at 93.0402 180.975 0)
+    (property "Value" "15F" (id 1) (at 95.0722 178.308 0)
+      (effects (font (size 1.27 1.27)) (justify left))
+    )
+    (property "Footprint" "Heliograph:SCCT30E156SRB" (id 2) (at 93.0402 180.975 0)
       (effects (font (size 1.27 1.27)) hide)
     )
@@
       (effects (font (size 1.27 1.27)) hide)
     )
-    (property "Part" "SCCT20E106SRB" (id 4) (at 92.075 177.165 0)
+    (property "Part" "SCCT30E156SRB" (id 4) (at 92.075 177.165 0)
       (effects (font (size 1.27 1.27)) hide)
     )
@@
     )
     (path "/00000000-0000-0000-0000-000061be4ac8"
-      (reference "C14") (unit 1) (value "10F") (footprint "Veridian-Library-KiCad:SCCT20E106SRB")
+      (reference "C14") (unit 1) (value "15F") (footprint "Heliograph:SCCT30E156SRB")
     )
     (path "/00000000-0000-0000-0000-000061b114b5"
@@
     )
     (path "/00000000-0000-0000-0000-000061bf4258"
-      (reference "C17") (unit 1) (value "10F") (footprint "Veridian-Library-KiCad:SCCT20E106SRB")
+      (reference "C17") (unit 1) (value "15F") (footprint "Heliograph:SCCT30E156SRB")
     )
     (path "/00000000-0000-0000-0000-000061cdbae3"
