File: PCB/PCBv1.2/SolarGPS.kicad_pcb (KiCad board)
At the start: 2 copper layers, 75 x 27 mm, 58 parts, among them J1 Conn_01x10_Female, J2 Solar1+, J3 GND, J4 Conn_02x03_Odd_Even, J5 Solar2+, J6 GND, J7 Screw_Terminal_01x01, J8 Conn_01x04_Male, U1 STM32L011G3Ux, U2 MAX-M10Q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

Commit message: Tweak Grounding
Routing:
- net Net-(D1-Pad2): track 52.5 -> 52.9 mm, vias 1 -> 2
Changed lines of the file:
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@@
   (segment (start 60.8 50.65) (end 59.8 51.65) (width 0.2) (layer "B.Cu") (net 60))
   (segment (start 59.8 53.45) (end 60.45 54.1) (width 0.2) (layer "B.Cu") (net 60))
+  (segment (start 108.52452 75.4) (end 110 76.87548) (width 0.2) (layer "F.Cu") (net 61))
+  (segment (start 102.5 75.1) (end 102.8 75.4) (width 0.2) (layer "F.Cu") (net 61))
   (segment (start 101.8 56.2) (end 101.9 56.3) (width 0.2) (layer "F.Cu") (net 61))
+  (segment (start 102.8 75.4) (end 108.52452 75.4) (width 0.2) (layer "F.Cu") (net 61))
   (segment (start 76.35 56.2) (end 101.8 56.2) (width 0.2) (layer "F.Cu") (net 61))
   (via (at 101.9 56.3) (size 0.6) (drill 0.3) (layers "F.Cu" "B.Cu") (net 61))
-  (segment (start 108.9 75.9) (end 109.82548 76.82548) (width 0.2) (layer "B.Cu") (net 61))
-  (segment (start 101.9 56.3) (end 101.9 74.25) (width 0.2) (layer "B.Cu") (net 61))
-  (segment (start 101.9 74.25) (end 103.55 75.9) (width 0.2) (layer "B.Cu") (net 61))
-  (segment (start 103.55 75.9) (end 108.9 75.9) (width 0.2) (layer "B.Cu") (net 61))
+  (via (at 102.5 75.1) (size 0.6) (drill 0.3) (layers "F.Cu" "B.Cu") (net 61))
+  (segment (start 102.5 75.1) (end 101.9 74.5) (width 0.2) (layer "B.Cu") (net 61))
+  (segment (start 101.9 74.5) (end 101.9 56.3) (width 0.2) (layer "B.Cu") (net 61))
   (segment (start 100.15 54.25) (end 103.45 50.95) (width 0.2) (layer "F.Cu") (net 62))
   (segment (start 103.45 50.95) (end 109.05 50.95) (width 0.2) (layer "F.Cu") (net 62))
   (segment (start 76.35 54.25) (end 100.15 54.25) (width 0.2) (layer "F.Cu") (net 62))
   (segment (start 109.05 50.95) (end 109.82548 50.17452) (width 0.2) (layer "F.Cu") (net 62))
-  (segment (start 69.026894 72.351786) (end 68.52868 72.85) (width 0.2) (layer "F.Cu") (net 63))
-  (segment (start 66.95 72.6) (end 60.825 72.6) (width 0.2) (layer "F.Cu") (net 63))
-  (segment (start 67.2 72.85) (end 66.95 72.6) (width 0.2) (layer "F.Cu") (net 63))
+  (segment (start 68.77868 72.6) (end 60.825 72.6) (width 0.2) (layer "F.Cu") (net 63))
+  (segment (start 69.026894 72.351786) (end 68.77868 72.6) (width 0.2) (layer "F.Cu") (net 63))
   (segment (start 60.825 72.6) (end 59.95 73.475) (width 0.2) (layer "F.Cu") (net 63))
-  (segment (start 68.52868 72.85) (end 67.2 72.85) (width 0.2) (layer "F.Cu") (net 63))
   (segment (start 57.99 72.76) (end 56.801 72.76) (width 0.2) (layer "F.Cu") (net 65))
   (segment (start 56.801 72.76) (end 56.801 74.03) (width 0.2) (layer "F.Cu") (net 65))

Commit message: Rebuild PCB1.2 and submit for build
Parts:
- J7: moved to F.Cu
- moved C18 2.64 mm to (50.9, 74.9), turned to 90 degrees
- moved C17 1.20 mm to (59.0, 63.5)
- moved C7 0.50 mm to (56.9, 60.4)
- turned J7 to -90 degrees
Routing:
- net RESET: track 19.7 -> 22.5 mm
- net VBATMID: track 61.2 -> 62.4 mm
- net VDD: track 154.9 -> 156.0 mm
- net GND: vias 62 -> 61
Other:
- board text added: "V1.2"
- board text removed: "V1.1"
