File: PCB/PCBv1.4/SolarGPS.kicad_pcb (KiCad board)
At the start: 2 copper layers, 80 x 32 mm, 49 parts, among them J1 Conn_01x24_Female, J2 GND, J3 GND, J4 AVR-ISP-6, J5 Solar2+, J6 Solar1+, J7 Screw_Terminal_01x01, J8 Conn_01x04_Male, Q1 Q_NMOS_GSD, U1 MAX40200AUK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

Commit message: Add demo code
Routing:
- net unconnected-(U4-Pad9): track 0.00 -> 2.21 mm
- net unconnected-(U3-Pad9): track 2.21 -> 0.00 mm
Changed lines of the file:
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@@
   (segment (start 87.7375 72.8625) (end 88.6 72) (width 0.2) (layer "B.Cu") (net 68))
   (segment (start 88.6 72) (end 89.55 72) (width 0.2) (layer "B.Cu") (net 68))
-  (segment (start 82.8625 76.65) (end 81.9125 77.6) (width 0.2) (layer "B.Cu") (net 71))
-  (segment (start 81.9125 77.6) (end 81.05 77.6) (width 0.2) (layer "B.Cu") (net 71))
+  (segment (start 82.8625 76.65) (end 81.9125 77.6) (width 0.2) (layer "B.Cu") (net 72))
+  (segment (start 81.9125 77.6) (end 81.05 77.6) (width 0.2) (layer "B.Cu") (net 72))
   (zone (net 1) (net_name "GND") (layers F&B.Cu) (hatch edge 0.508)
     (connect_pads (clearance 0.2))
