File: PCB/PCBv1.4/SolarGPS.kicad_sch (KiCad schematic)
At the start: 45 parts, among them J1 Conn_01x24_Female, J2 GND, J3 GND, J4 Conn_02x03_Odd_Even, J5 Solar2+, J6 Solar1+, J7 Screw_Terminal_01x01, J8 Conn_01x04_Male, Q1 Q_NMOS_GSD, U1 STM32L011G4Ux, U2 MAX-M10Q, U6 LIS3DH, Y1 32.768

Commit message: Update 1.4 BOM
Parts:
- removed C11: 1uF, Capacitor_SMD:C_0603_1608Metric, symbol Device:C_Small
- removed C12: 4.7uF, Capacitor_SMD:C_0805_2012Metric, symbol Device:C_Small
- C5: footprint Capacitor_SMD:C_0603_1608Metric -> Capacitor_SMD:C_0805_2012Metric
- C8: value 30F -> 25F; footprint Heliograph:SCCT30E156SRB -> Heliograph:TPLC3R8-25MR8X20; Part (none) -> TPLC-3R8/25MR8X20
- R1: value 91k -> 1M
- R2: value 149 -> 120
Connections:
- net LED: now also U1.28 (PB7); no longer U1.12 (PA6)
- net CORE: now reaches C16.1, J1.18 (Pin_18)
- net VBAT_SENSE: no longer names the net of U1.11 (PA5)
- no-connect marks 19 -> 22
Other:
- note added: "Super Cap: 3.8-2.20V GPS: 3.6-2.70V LIS3DH: 3.6-1.80V STM32G0: 3.6-1.65V DISP: 3.7-2.20V ---------- SYS: 3.6-2.70V"
- note removed: "ANALOG"
- moved on the sheet: AE1, C1, C5, R7, U2

Commit message: firmware stuff
Parts:
- removed C15, C16, C2, C22, C3, C6: 1uF, Capacitor_SMD:C_0603_1608Metric, symbol Device:C_Small
- removed C8: 25F, Heliograph:TPLC3R8-25MR8X20, symbol Device:CP
- removed D4, D5, D6: B0530WS, Diode_SMD:D_SOD-323_HandSoldering, symbol Device:D_Schottky_Small
- removed J1: Conn_01x24_Female, Heliograph:ER-CON24HT-1, symbol Connector:Conn_01x24_Female
- removed L1: 47uH, Inductor_SMD:L_Taiyo-Yuden_NR-40xx, symbol Device:L_Small
- removed Q1: Q_NMOS_GSD, Package_TO_SOT_SMD:SOT-23, symbol Device:Q_NMOS_GSD
- removed R2: 120, Resistor_SMD:R_0603_1608Metric, symbol Device:R_Small
- removed U1: STM32L011G4Ux, Package_DFN_QFN:QFN-28_4x4mm_P0.5mm, symbol MCU_ST_STM32L0:STM32L011G4Ux
- added C11, C8: 1uF, Capacitor_SMD:C_0603_1608Metric, symbol Device:C_Small
- added C13: 4.7uF, Capacitor_SMD:C_0805_2012Metric, symbol Device:C_Small
- added C14: 25F, Heliograph:TPLC3R8-25MR8X20, symbol Device:CP
- added C23: 10nF, Capacitor_SMD:C_0603_1608Metric, symbol Device:C_Small
- added J1: Conn_01x10_Female, Margo_Lib:LS013B7DH03, symbol Connector:Conn_01x10_Female
- added L2: 0.47uH, Inductor_SMD:L_0806_2016Metric, symbol Device:L_Small
- added R12, R13: 1M, Resistor_SMD:R_0603_1608Metric, symbol Device:R_Small
- added R4, R?: 432k, Resistor_SMD:R_0603_1608Metric, symbol Device:R_Small
- added R5: 91k, Resistor_SMD:R_0603_1608Metric, symbol Device:R_Small
- added U1: STM32L011G3Ux, Package_DFN_QFN:QFN-28_4x4mm_P0.5mm, symbol MCU_ST_STM32L0:STM32L011G3Ux
- added U7: TPS63802, Margo_Lib:VREG_TPS63802DLAR, symbol SolarGPS-rescue:TPS63802-VeridianDesigns
- C18: value 1uF -> 10nF
- C5: value 22uF -> 10nF; footprint Capacitor_SMD:C_0805_2012Metric -> Capacitor_SMD:C_0603_1608Metric; Part GRM187R61A226ME15 -> (none)
- C7: value 1uF -> 47uF; footprint Capacitor_SMD:C_0603_1608Metric -> Capacitor_SMD:C_1206_3216Metric
- D1, D3: value B0530WS -> Schottky
- J2: value GND -> Solar1+
- J6: value Solar1+ -> GND
- R1: value 1M -> 91k
- R3: value 2.2 -> 390
Connections:
- net RESE is gone; now on an unnamed net: R3.2
- net SWDCLK is gone; now on net SWO: J4.4 (Pin_4)
- net VGH is gone; now on net GND: C20.1
- net VGL is gone; now on net GND: C21.2
- net VSH2 is gone; now on net GND: C9.1
- net BOOT0: now also U1.1 (PB9)
- net DISP_CS: now also J1.3 (Pin_3), U1.23 (PA15)
- net GND: now also C5.1, J6.1 (Pin_1), C11.2, C13.2, C14.2, C23.1, C8.1, R13.1, R5.1, U1.16 (VSS), U1.27 (PB6), U7.2 (MODE), U7.3 (AGND), U7.8 (GND); no longer C20.2, C21.1, C5.2, C9.2, J2.1 (Pin_1), R3.1
- net GPS_EXINT: now also U1.15 (PB1)
- net GPS_UART_MISO: now also U1.6 (PA0)
- net GPS_UART_MOSI: now also U1.8 (PA2)
- net LED: now also R3.1
- net LIS_CS: now also U1.18 (PA8)
- net LIS_INT: now also U1.28 (PB7)
- net RESET: now also U1.4 (NRST)
- net SPI_CLK: now also J1.1 (Pin_1), U1.24 (PB3)
- net SPI_MISO: now also U1.25 (PB4)
- net SPI_MOSI: now also J1.2 (Pin_2), U1.26 (PB5)
- net SWDIO: now also U1.21 (PA13)
- net VDD: now also C21.1, C5.2, C9.2, C11.1, C13.1, J1.6 (Pin_6), J1.7 (Pin_7), J1.8 (Pin_8), R4.2, R?.2, U1.17 (VDD), U1.5 (VDDA), U7.6 (VOUT); no longer C5.1, D1.1 (K), D3.1 (K)
- net at C4.1, Y1.2: now also U1.2 (PC14)
- net at C10.1, Y1.1: now also U1.3 (PC15)
- net at D3.2 (A): now also J2.1 (Pin_1); no longer J6.1 (Pin_1)
- net SWO: now reaches J4.6 (Pin_6)
- net SWO: now also U1.22 (PA14)
- new net: J1.10 (Pin_10), J1.9 (Pin_9)
- new net: R4.1, R5.2, U7.4 (FB)
- new net: L2.2, U7.7 (L2)
- new net: L2.1, U7.9 (L1)
- new net DISP_EN: C20.2, J1.5 (Pin_5), U1.20 (PA10)
- new net EXTCOMIN: J1.4 (Pin_4), U1.19 (PA9)
- new net PG: R?.1, U7.5 (PG)
- new net VBAT: C14.1, C8.2, D1.1 (K), D3.1 (K), R12.2, U7.10 (VIN)
- new net VBAT_EN: U1.11 (PA5)
- new net VBAT_SENSE: C23.2, R12.1, R13.2, U7.1 (EN)
- no-connect marks 22 -> 15
Other:
- note added: "ANALOG"
- note added: "VOUT = 2.87"
- note removed: "ER-EPD0154-2R"
- note removed: "Super Cap: 3.8-2.20V GPS: 3.6-2.70V LIS3DH: 3.6-1.80V STM32G0: 3.6-1.65V DISP: 3.7-2.20V ---------- SYS: 3.6-2.70V"
- note removed: "VCI: 2.2 to 3.7V VDDIO: Connect to VCI VDD: 1.8V, regulate from VCI supply"
- moved on the sheet: AE1, C1, C10, C25, C26, C4, C9, D2, J4, J7, R3, R7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
