File: PCB/PCBv1.5/SolarGPS.kicad_sch (KiCad schematic)
At the start: 46 parts, among them J1 Conn_01x24_Female, J2 GND, J3 GND, J4 AVR-ISP-6, J5 Solar2+, J6 Solar1+, J7 Screw_Terminal_01x01, J8 Conn_01x04_Male, Q1 Q_NMOS_GSD, Q2 Q_NMOS_GSD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

Commit message: Version 1.4
Parts:
- removed C10: 11pF, Capacitor_SMD:C_0603_1608Metric, symbol Device:C_Small
- removed C17, C18: 1uF, Capacitor_SMD:C_0603_1608Metric, symbol Device:C_Small
- removed J4: AVR-ISP-6, Connector_PinHeader_2.54mm:PinHeader_2x03_P2.54mm_Vertical, symbol Connector:AVR-ISP-6
- removed Q2: Q_NMOS_GSD, Package_TO_SOT_SMD:SOT-23, symbol Device:Q_NMOS_GSD
- removed R1: 1M, Resistor_SMD:R_0603_1608Metric, symbol Device:R_Small
- removed U3: ATmega328PB-M, Package_DFN_QFN:QFN-32-1EP_5x5mm_P0.5mm_EP3.1x3.1mm, symbol MCU_Microchip_ATmega:ATmega328PB-M
- removed U4: ATmega328PB-A, Package_QFP:TQFP-32_7x7mm_P0.8mm, symbol MCU_Microchip_ATmega:ATmega328PB-A
- removed Y1: 32.768, Crystal:Crystal_SMD_3215-2Pin_3.2x1.5mm, symbol Device:Crystal
- added J4: Conn_01x03_Female, Connector_PinHeader_2.00mm:PinHeader_1x03_P2.00mm_Vertical, symbol Connector:Conn_01x03_Female
- added U1: MAX40200AUK, Package_TO_SOT_SMD:SOT-23-5, symbol Analog_Switch:MAX40200AUK
- added U3: ATtiny3216-M, Package_DFN_QFN:VQFN-20-1EP_3x3mm_P0.4mm_EP1.7x1.7mm, symbol MCU_Microchip_ATtiny:ATtiny3216-M
- C19: value 1uF -> 1nF
- C4: value 11pF -> 1uF
- C5: value 47uF -> 1uF; footprint Capacitor_SMD:C_0805_2012Metric -> Capacitor_SMD:C_0603_1608Metric; Part GRM187R61A226ME15 -> (none)
- D2: Part LS R976-NR-1 -> LTST-S220KRKT
- Q1: Part NX3008NBK -> DMN3730U-7
- R2: value 149 -> 100
Connections:
- net AREF is gone; now on net VBAT: C19.1
- net XTAL2 is gone; now on net GND: C4.1
- net DISP_BUSY: now also U3.13 (PB1)
- net DISP_CS: now also U3.18 (PC3)
- net DISP_DC: now also U3.8 (PA7)
- net DISP_RES#: now also U3.16 (PC1)
- net GND: now also C14.2, C19.2, C5.1, C8.2, D2.1 (K), J2.1 (Pin_1), J3.1 (Pin_1), J4.3 (Pin_3), U1.2 (GND), U3.21 (GND), U3.3 (GND); no longer C5.2
- net GPS_EXINT: now also U3.10 (PB4); no longer R7.2
- net GPS_UART_MISO: now also U3.12 (PB2)
- net GPS_UART_MOSI: now also U3.11 (PB3)
- net LED: now also U3.15 (PC0)
- net LIS_CS: now also U3.6 (PA5)
- net LIS_INT: now also U3.7 (PA6)
- net SPI_CLK: now also U3.20 (PA1)
- net SPI_MISO: now also U3.1 (PA2)
- net SPI_MOSI: now also U3.2 (PA3)
- net VBAT: now also C4.2, J4.1 (Pin_1), U1.1 (VDD), U3.4 (VCC); no longer C5.1, U2.6 (V_BCKP), U2.7 (VCC_IO), U2.8 (VCC)
- removed net GNDPWR: C14.2, C19.2, C4.2, C8.2, D2.1 (K), J2.1 (Pin_1), J3.1 (Pin_1)
- new net GPSVDD: C5.2, U1.5 (OUT), U2.6 (V_BCKP), U2.7 (VCC_IO), U2.8 (VCC)
- new net GPS_EN: R7.2, U1.3 (EN), U3.14 (PB0)
- new net UPDI: J4.2 (Pin_2), U3.19 (~{RESET}/PA0)
- no-connect marks 24 -> 18
Other:
- moved on the sheet: AE1, C1, C14, C19, C21, D2, J3, J8, R2, R7, U2

Commit message: tweak pcb1.5
Parts:
- added R1: 1M, Resistor_SMD:R_0603_1608Metric, symbol Device:R_Small
Connections:
- net GND: now also R1.1
- net at D2.2 (A), R2.1: now also R1.2
- no-connect marks 18 -> 19
Other:
- note added: "VCC Range: 2.2-3.6"
- moved on the sheet: C14, C19, D2, J4, R2

Commit message: Some dumb changes
Parts:
- removed C15, C16, C20, C21, C22, C4, C6, C9: 1uF, Capacitor_SMD:C_0603_1608Metric, symbol Device:C_Small
- removed D4, D5, D6: B0530WS-TP, Diode_SMD:D_SOD-323, symbol Device:D_Schottky_Small
- removed J1: Conn_01x24_Female, Heliograph:ER-CON24HT-1, symbol Connector:Conn_01x24_Female
- removed J4: Conn_01x03_Female, Connector_PinHeader_2.00mm:PinHeader_1x03_P2.00mm_Vertical, symbol Connector:Conn_01x03_Female
- removed L1: 47uH, Inductor_SMD:L_Taiyo-Yuden_NR-40xx, symbol Device:L_Small
- removed Q1: Q_NMOS_GSD, Package_TO_SOT_SMD:SOT-23, symbol Device:Q_NMOS_GSD
- removed R1, R7: 1M, Resistor_SMD:R_0603_1608Metric, symbol Device:R_Small
- removed R3: 2.2, Resistor_SMD:R_0603_1608Metric, symbol Device:R_Small
- removed U1: MAX40200AUK, Package_TO_SOT_SMD:SOT-23-5, symbol Analog_Switch:MAX40200AUK
- removed U3: ATtiny3216-M, Package_DFN_QFN:VQFN-20-1EP_3x3mm_P0.4mm_EP1.7x1.7mm, symbol MCU_Microchip_ATtiny:ATtiny3216-M
- added C?: 1uF, Capacitor_SMD:C_0603_1608Metric, symbol Device:C_Small
- added C? (x2): 11pF, Capacitor_SMD:C_0603_1608Metric, symbol Device:C_Small
- added J1: Conn_01x10_Female, Heliograph:LS013B7DH03, symbol Connector:Conn_01x10_Female
- added J?: Conn_02x03_Odd_Even, symbol Connector_Generic:Conn_02x03_Odd_Even
- added JP1: Jumper_3_Bridged12, symbol Jumper:Jumper_3_Bridged12
- added U?: STM32L433CCUx, Package_DFN_QFN:QFN-48-1EP_7x7mm_P0.5mm_EP5.6x5.6mm, symbol MCU_ST_STM32L4:STM32L433CCUx
- added Y?: 32.768, Crystal:Crystal_SMD_3215-2Pin_3.2x1.5mm, symbol Device:Crystal
- C19: value 1nF -> 1uF
Connections:
- net GPSVDD is gone; now on net VBAT: C5.2, U2.6 (V_BCKP), U2.7 (VCC_IO), U2.8 (VCC)
- net VCOM is gone; now on net GND: C2.1
- net VSL is gone; now on net GND: C3.1
- net GND: now also C?.2, C?.2, C?.2, J1.10 (Pin_10), J1.9 (Pin_9), J?.5 (Pin_5), JP1.3 (B); no longer C2.2, C3.2
- net GPS_UART_MISO: now also U?.13 (PA3)
- net GPS_UART_MOSI: now also U?.12 (PA2)
- net SPI_CLK: now also J1.1 (Pin_1), U?.11 (PA1)
- net SPI_MISO: now also U?.16 (PA6)
- net SPI_MOSI: now also J1.2 (Pin_2), U?.17 (PA7)
- net VBAT: now also C2.2, C3.2, C?.1, J1.6 (Pin_6), J1.7 (Pin_7), J?.1 (Pin_1), JP1.1 (A), U?.1 (VBAT), U?.24 (VDD), U?.48 (VDD), U?.9 (VDDA)
- new net DISPCS: J1.3 (Pin_3)
- new net DISPEN: J1.5 (Pin_5)
- new net EXTCOMIN: J1.4 (Pin_4)
- new net EXTSEL: J1.8 (Pin_8), JP1.2 (C)
- new net SWCLK: J?.4 (Pin_4), U?.37 (PA14)
- new net SWDIO: J?.2 (Pin_2), U?.34 (PA13)
- new net SWO: J?.6 (Pin_6), U?.39 (PB3)
- new net XTAL1: C?.1, U?.3 (PC14), Y?.1
- new net XTAL2: C?.1, U?.2 (PC13), Y?.2
- new net nRESET: J?.3 (Pin_3), U?.7 (NRST)
- no-connect marks 19 -> 12
Other:
- note added: "VMAX: 0-3.6"
- note removed: "ER-EPD0154-2R"
- note removed: "VCI: 2.2 to 3.7V VDDIO: Connect to VCI VDD: 1.8V, regulate from VCI supply"
- moved on the sheet: C14, C19, C5, D2, R2
