File: PCB/PCBv1.5/SolarGPS.kicad_pcb (KiCad board)
At the start: 2 copper layers, 80 x 32 mm, 40 parts, among them J1 Conn_01x24_Female, J2 GND, J3 GND, J4 Conn_01x03_Female, J5 Solar2+, J6 Solar1+, J7 Screw_Terminal_01x01, J8 Conn_01x04_Male, Q1 Q_NMOS_GSD, U1 MAX40200AUK, U2 MAX-M10Q, U3 ATtiny3216-M, U6 LIS3DH

Commit message: tweak pcb1.5
Parts:
- added R1: 1M, Resistor_SMD:R_0603_1608Metric, F.Cu at (117.4, 62.7)
Routing:
- net Net-(R2-Pad1): track 1.54 -> 2.94 mm
- net GPS_UART_MOSI: track 56.9 -> 56.8 mm, vias 2 -> 1
Changed lines of the file:
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@@
   (net 4 "GPS_UART_MOSI")
   (net 5 "GPS_UART_MISO")
-  (net 6 "Net-(D2-Pad2)")
+  (net 6 "Net-(R2-Pad1)")
   (net 7 "LED")
   (net 8 "/GPS_RF")
@@
       (net 1 "GND") (pinfunction "K") (pintype "passive"))
     (pad "2" smd roundrect locked (at 0.9375 0 90) (size 0.975 1.4) (layers "F.Cu" "F.Paste" "F.Mask") (roundrect_rratio 0.25)
-      (net 6 "Net-(D2-Pad2)") (pinfunction "A") (pintype "passive"))
+      (net 6 "Net-(R2-Pad1)") (pinfunction "A") (pintype "passive"))
     (model "${KISYS3DMOD}/Diode_SMD.3dshapes/D_0805_2012Metric.wrl"
       (offset (xyz 0 0 0))
@@
       (net 44 "DISP_DC") (pinfunction "PA7") (pintype "bidirectional"))
     (pad "9" smd roundrect (at 0.4 1.45) (size 0.2 0.8) (layers "F.Cu" "F.Paste" "F.Mask") (roundrect_rratio 0.25)
-      (net 55 "unconnected-(U3-Pad9)") (pinfunction "PB5") (pintype "bidirectional"))
+      (net 55 "unconnected-(U3-Pad9)") (pinfunction "PB5") (pintype "bidirectional+no_connect"))
     (pad "10" smd custom (at 0.8 1.45) (size 0.143431 0.143431) (layers "F.Cu" "F.Paste" "F.Mask")
       (net 2 "GPS_EXINT") (pinfunction "PB4") (pintype "bidirectional")
@@
     )
   )
+  (footprint "Resistor_SMD:R_0603_1608Metric" (layer "F.Cu")
+    (at 117.4 62.7 -90)
+    (descr "Resistor SMD 0603 (1608 Metric), square (rectangular) end terminal, IPC_7351 nominal, (Body size source: IPC-SM-782 page 72, https://www.pcb-3d.com/wordpress/wp-content/uploads/ipc-sm-782a_amendment_1_and_2.pdf), generated with kicad-footprint-generator")
+    (tags "resistor")
+    (property "Sheetfile" "SolarGPS.kicad_sch")
+    (property "Sheetname" "")
+    (attr smd)
+    (fp_text reference "R1" (at 0 -1.43 90) (layer "F.SilkS")
+      (effects (font (size 1 1) (thickness 0.15)))
+    )
+    (fp_text value "1M" (at 0 1.43 90) (layer "F.Fab")
+      (effects (font (size 1 1) (thickness 0.15)))
+    )
+    (fp_text user "${REFERENCE}" (at 0 0 90) (layer "F.Fab")
+      (effects (font (size 0.4 0.4) (thickness 0.06)))
+    )
+    (fp_line (start -0.237258 0.5225) (end 0.237258 0.5225) (layer "F.SilkS") (width 0.12))
+    (fp_line (start -0.237258 -0.5225) (end 0.237258 -0.5225) (layer "F.SilkS") (width 0.12))
+    (fp_line (start 1.48 -0.73) (end 1.48 0.73) (layer "F.CrtYd") (width 0.05))
+    (fp_line (start -1.48 0.73) (end -1.48 -0.73) (layer "F.CrtYd") (width 0.05))
+    (fp_line (start -1.48 -0.73) (end 1.48 -0.73) (layer "F.CrtYd") (width 0.05))
+    (fp_line (start 1.48 0.73) (end -1.48 0.73) (layer "F.CrtYd") (width 0.05))
+    (fp_line (start -0.8 0.4125) (end -0.8 -0.4125) (layer "F.Fab") (width 0.1))
+    (fp_line (start -0.8 -0.4125) (end 0.8 -0.4125) (layer "F.Fab") (width 0.1))
+    (fp_line (start 0.8 0.4125) (end -0.8 0.4125) (layer "F.Fab") (width 0.1))
+    (fp_line (start 0.8 -0.4125) (end 0.8 0.4125) (layer "F.Fab") (width 0.1))
+    (pad "1" smd roundrect (at -0.825 0 270) (size 0.8 0.95) (layers "F.Cu" "F.Paste" "F.Mask") (roundrect_rratio 0.25)
+      (net 1 "GND") (pintype "passive"))
+    (pad "2" smd roundrect (at 0.825 0 270) (size 0.8 0.95) (layers "F.Cu" "F.Paste" "F.Mask") (roundrect_rratio 0.25)
+      (net 6 "Net-(R2-Pad1)") (pintype "passive"))
+    (model "${KICAD6_3DMODEL_DIR}/Resistor_SMD.3dshapes/R_0603_1608Metric.wrl"
+      (offset (xyz 0 0 0))
+      (scale (xyz 1 1 1))
+      (rotate (xyz 0 0 0))
+    )
+  )
   (footprint "Capacitor_SMD:C_0603_1608Metric" (layer "F.Cu")
     (at 57 67.45 180)
@@
     (fp_line (start 0.8 0.4125) (end -0.8 0.4125) (layer "F.Fab") (width 0.1))
     (pad "1" smd roundrect (at -0.825 0 90) (size 0.8 0.95) (layers "F.Cu" "F.Paste" "F.Mask") (roundrect_rratio 0.25)
-      (net 6 "Net-(D2-Pad2)") (pintype "passive"))
+      (net 6 "Net-(R2-Pad1)") (pintype "passive"))
     (pad "2" smd roundrect (at 0.825 0 90) (size 0.8 0.95) (layers "F.Cu" "F.Paste" "F.Mask") (roundrect_rratio 0.25)
       (net 7 "LED") (pintype "passive"))
@@
   (via (at 111.6 79) (size 0.6) (drill 0.3) (layers "F.Cu" "B.Cu") (net 2))
   (via (at 124.6 77.4) (size 0.6) (drill 0.3) (layers "F.Cu" "B.Cu") (net 2))
-  (segment (start 112.6 78) (end 113.2 77.4) (width 0.2) (layer "B.Cu") (net 2))
-  (segment (start 113.2 77.4) (end 124.6 77.4) (width 0.2) (layer "B.Cu") (net 2))
-  (segment (start 111.6 79) (end 112.6 78) (width 0.2) (layer "B.Cu") (net 2))
+  (segment (start 112.4 78.2) (end 123.8 78.2) (width 0.2) (layer "B.Cu") (net 2))
+  (segment (start 111.6 79) (end 112.4 78.2) (width 0.2) (layer "B.Cu") (net 2))
+  (segment (start 123.8 78.2) (end 124.6 77.4) (width 0.2) (layer "B.Cu") (net 2))
   (segment (start 64.65 65.75) (end 73.6 74.7) (width 0.2) (layer "F.Cu") (net 3))
   (segment (start 73.6 74.7) (end 73.6 76.65) (width 0.2) (layer "F.Cu") (net 3))
@@
   (segment (start 109.2 78.9) (end 110.3 77.8) (width 0.2) (layer "F.Cu") (net 4))
   (segment (start 122.35 77.75) (end 119 74.4) (width 0.2) (layer "F.Cu") (net 4))
-  (segment (start 110.2 73.715) (end 112.625 71.29) (width 0.2) (layer "F.Cu") (net 4))
   (segment (start 115.735 74.4) (end 112.625 71.29) (width 0.2) (layer "F.Cu") (net 4))
-  (segment (start 110.2 75.2) (end 110.2 73.715) (width 0.2) (layer "F.Cu") (net 4))
   (via (at 110.3 77.8) (size 0.6) (drill 0.3) (layers "F.Cu" "B.Cu") (net 4))
-  (via (at 110.2 75.2) (size 0.6) (drill 0.3) (layers "F.Cu" "B.Cu") (net 4))
-  (segment (start 110.3 75.3) (end 110.2 75.2) (width 0.2) (layer "B.Cu") (net 4))
-  (segment (start 110.3 77.8) (end 110.3 75.3) (width 0.2) (layer "B.Cu") (net 4))
+  (segment (start 110.3 73.615) (end 112.625 71.29) (width 0.2) (layer "B.Cu") (net 4))
+  (segment (start 110.3 77.8) (end 110.3 73.615) (width 0.2) (layer "B.Cu") (net 4))
+  (segment (start 110.37 73.83) (end 112.625 73.83) (width 0.2) (layer "F.Cu") (net 5))
   (segment (start 121.25 77.45) (end 121.25 78.95) (width 0.2) (layer "F.Cu") (net 5))
-  (segment (start 107.955 78.5) (end 112.625 73.83) (width 0.2) (layer "F.Cu") (net 5))
   (segment (start 113.795 75) (end 118.8 75) (width 0.2) (layer "F.Cu") (net 5))
-  (segment (start 75.05 78.5) (end 107.955 78.5) (width 0.2) (layer "F.Cu") (net 5))
   (segment (start 112.625 73.83) (end 113.795 75) (width 0.2) (layer "F.Cu") (net 5))
+  (segment (start 105.7 78.5) (end 110.37 73.83) (width 0.2) (layer "F.Cu") (net 5))
   (segment (start 118.8 75) (end 121.25 77.45) (width 0.2) (layer "F.Cu") (net 5))
+  (segment (start 75.05 78.5) (end 105.7 78.5) (width 0.2) (layer "F.Cu") (net 5))
   (segment (start 116 63.525) (end 116 65.0625) (width 0.2) (layer "F.Cu") (net 6))
+  (segment (start 116 63.525) (end 117.4 63.525) (width 0.2) (layer "F.Cu") (net 6))
   (segment (start 75.05 77.3) (end 75.85 76.5) (width 0.2) (layer "F.Cu") (net 7))
   (segment (start 75.85 76.5) (end 99.7 76.5) (width 0.2) (layer "F.Cu") (net 7))

Commit message: Manufacture 1.5 PCB
Parts:
- removed C20, C21, C22: 1uF, Capacitor_SMD:C_0603_1608Metric
- removed D4, D5, D6: B0530WS-TP, Diode_SMD:D_SOD-323
- removed Q1: Q_NMOS_GSD, Package_TO_SOT_SMD:SOT-23
- removed R7: 1M, Resistor_SMD:R_0603_1608Metric
- added C10: 47uF, Capacitor_SMD:C_1206_3216Metric, F.Cu at (57.2, 55.1)
- added C11: 4.7uF, Capacitor_SMD:C_0805_2012Metric, F.Cu at (71.2, 53.2)
- added C12: 47uF, Capacitor_SMD:C_1206_3216Metric, F.Cu at (57.2, 57.5)
- added C13: 11pF, Capacitor_SMD:C_0603_1608Metric, F.Cu at (57.4, 79.0)
- added C7: 10nF, Capacitor_SMD:C_0603_1608Metric, F.Cu at (67.2, 58.6)
- added ROK1: 6.49M, Resistor_SMD:R_0603_1608Metric, F.Cu at (62.1, 58.1)
- added ROK2: 5.36M, Resistor_SMD:R_0603_1608Metric, F.Cu at (61.3, 56.0)
- added ROK3: 1M, Resistor_SMD:R_0603_1608Metric, F.Cu at (61.3, 53.2)
- added ROV1: 6.49M, Resistor_SMD:R_0603_1608Metric, F.Cu at (60.6, 50.7)
- added ROV2: 6.49M, Resistor_SMD:R_0603_1608Metric, F.Cu at (62.7, 51.5)
- added Y1: 32.768, Crystal:Crystal_SMD_3215-2Pin_3.2x1.5mm, F.Cu at (59.9, 77.9)
- C15: value 1uF -> 11pF
- C19: value 1nF -> 1uF
- C4: value 1uF -> 4.7uF; footprint Capacitor_SMD:C_0603_1608Metric -> Capacitor_SMD:C_0805_2012Metric
- C6, C9: value 1uF -> 10nF
- D1, D3: value B0530WS-TP -> Schottky; footprint Diode_SMD:D_SOD-323 -> Diode_SMD:D_SOD-323_HandSoldering
- J1: value Conn_01x24_Female -> Conn_01x10_Female; footprint Heliograph:ER-CON24HT-1 -> Heliograph:LS013B7DH03
- J2: value GND -> Solar2+; moved to F.Cu
- J3: value GND -> Solar1+; moved to F.Cu
- J4: value Conn_01x03_Female -> GND; footprint Connector_PinHeader_2.00mm:PinHeader_1x03_P2.00mm_Vertical -> Connector_PinHeader_2.54mm:PinHeader_1x01_P2.54mm_Vertical
- J5: value Solar2+ -> GND; moved to F.Cu
- J6: value Solar1+ -> Conn_02x03_Odd_Even; footprint Connector_PinHeader_2.54mm:PinHeader_1x01_P2.54mm_Vertical -> Connector:Tag-Connect_TC2030-IDC-NL_2x03_P1.27mm_Vertical; moved to F.Cu
- L1: value 47uH -> 22uH; footprint Inductor_SMD:L_Taiyo-Yuden_NR-40xx -> Heliograph:744031220
- R1: value 1M -> 100
- R3: value 2.2 -> 100
- U1: value MAX40200AUK -> BQ25505; footprint Package_TO_SOT_SMD:SOT-23-5 -> Package_DFN_QFN:QFN-20-1EP_3.5x3.5mm_P0.5mm_EP2x2mm
- U3: value ATtiny3216-M -> STM32L031G6Ux; footprint Package_DFN_QFN:VQFN-20-1EP_3x3mm_P0.4mm_EP1.7x1.7mm -> Package_DFN_QFN:QFN-28_4x4mm_P0.5mm
- moved J2 68.0 mm to (115.0, 52.0), turned to 0 degrees
- moved J3 67.2 mm to (115.0, 78.0), turned to 0 degrees
- moved J6 64.7 mm to (53.9, 73.4), turned to 0 degrees
- moved J5 61.0 mm to (54.0, 78.0), turned to 0 degrees
- moved R1 60.4 mm to (58.1, 74.1)
- moved U1 53.3 mm to (65.8, 54.4), turned to 180 degrees
- moved D1 46.5 mm to (75.0, 53.9), turned to 0 degrees
- moved D3 40.4 mm to (75.0, 55.8), turned to 0 degrees
- moved J4 29.5 mm to (55.0, 52.0), turned to 0 degrees
- moved R3 28.5 mm to (70.7, 78.3), turned to 0 degrees
- moved C6 19.7 mm to (69.1, 51.9), turned to 90 degrees
- moved C15 13.0 mm to (57.4, 77.7), turned to 180 degrees
- moved U3 12.1 mm to (62.6, 73.0), turned to 90 degrees
- moved C16 12.1 mm to (51.4, 76.8), turned to -90 degrees
- moved C3 11.8 mm to (61.9, 63.8), turned to 0 degrees
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Connections:
- C14 pad 1: VBAT -> VDD
- C15 pad 1: GND -> XTAL1
- C15 pad 2: VBAT -> GND
- C16 pad 1: Net-(C16-Pad1) -> VDD
- C19 pad 1: VBAT -> VDD
- C2 pad 1: /VCOM -> nRESET
- C26 pad 2: VBAT -> VDD
- C3 pad 1: /VSL -> GND
- C3 pad 2: GND -> VDD
- C4 pad 1: GND -> SOLAR+
- C4 pad 2: VBAT -> GND
- C5 pad 2: /GPSVDD -> VDD
- C6 pad 1: /VSH1 -> Net-(C6-Pad1)
- C9 pad 1: /VSH2 -> GND
- C9 pad 2: GND -> VBAT
- D1 pad 1: VBAT -> SOLAR+
- D2 pad 2: Net-(R2-Pad1) -> Net-(D2-Pad2)
- D3 pad 1: VBAT -> SOLAR+
- J1 pad 1: unconnected-(J1-Pad1) -> SPI_CLK
- J1 pad 10: DISP_RES# -> GND
- J1 pad 2: /GDR -> SPI_MOSI
- J1 pad 3: /RESE -> DISPCS
- J1 pad 4: unconnected-(J1-Pad4) -> EXTCOMIN
- J1 pad 5: /VSH2 -> DISPEN
- J1 pad 6: unconnected-(J1-Pad6) -> VDD
- J1 pad 7: unconnected-(J1-Pad7) -> VDD
- J1 pad 8: GND -> VDD
- J1 pad 9: DISP_BUSY -> GND
- J2 pad 1: GND -> Net-(D1-Pad2)
- J3 pad 1: GND -> Net-(D3-Pad2)
- J4 pad 1: VBAT -> GND
- J5 pad 1: Net-(D1-Pad2) -> GND
- J6 pad 1: Net-(D3-Pad2) -> VDD
- J8 pad 1: VBAT -> VDD
- L1 pad 1: VBAT -> SOLAR+
- L1 pad 2: Net-(C22-Pad1) -> /LBOOST
- R1 pad 1: GND -> Net-(R1-Pad1)
- R1 pad 2: Net-(R2-Pad1) -> GND
- R2 pad 1: Net-(R2-Pad1) -> Net-(D2-Pad2)
- R3 pad 1: GND -> Net-(R3-Pad1)
- R3 pad 2: /RESE -> SOLAR+
- U1 pad 1: VBAT -> GND
- U1 pad 2: GND -> SOLAR+
- U1 pad 3: GPS_EN -> VDD
- U1 pad 4: unconnected-(U1-Pad4) -> Net-(C6-Pad1)
- U1 pad 5: /GPSVDD -> GND
- U2 pad 6: /GPSVDD -> VDD
- U2 pad 7: /GPSVDD -> VDD
- U2 pad 8: /GPSVDD -> VDD
- U3 pad 1: SPI_MISO -> VDD
- U3 pad 10: GPS_EXINT -> LIS_CS
- U3 pad 11: GPS_UART_MOSI -> SPI_CLK
- U3 pad 12: GPS_UART_MISO -> SPI_MISO
- U3 pad 13: DISP_BUSY -> SPI_MOSI
- U3 pad 14: GPS_EN -> LIS_INT
- U3 pad 15: LED -> VBAT_OK
- U3 pad 16: DISP_RES# -> GND
- U3 pad 17: unconnected-(U3-Pad17) -> VDD
- U3 pad 18: DISP_CS -> DISPEN
- U3 pad 19: UPDI -> SWO
- U3 pad 2: SPI_MOSI -> XTAL1
- U3 pad 20: SPI_CLK -> DISPCS
- U3 pad 21: GND -> SWDIO
- U3 pad 3: GND -> XTAL2
- U3 pad 4: VBAT -> nRESET
- U3 pad 5: unconnected-(U3-Pad5) -> VDD
- U3 pad 6: LIS_CS -> Net-(R3-Pad1)
- U3 pad 7: LIS_INT -> GPS_EXINT
- U3 pad 8: DISP_DC -> GPS_UART_MOSI
- U3 pad 9: unconnected-(U3-Pad9) -> GPS_UART_MISO
- U6 pad 1: VBAT -> VDD
- U6 pad 14: VBAT -> VDD
Routing:
- net VDD: track 0.00 -> 172.4 mm, vias 0 -> 8
- net VBAT: track 148.7 -> 24.5 mm, vias 6 -> 2
- net Net-(D3-Pad2): track 2.12 -> 54.7 mm, vias 0 -> 1
- net GPS_EN: track 48.5 -> 0.00 mm
- net LED: track 47.3 -> 0.00 mm
- net Net-(D1-Pad2): track 2.12 -> 40.6 mm, vias 0 -> 1
- net SOLAR+: track 0.00 -> 34.3 mm, vias 0 -> 2
- net /VGL: track 27.0 -> 0.00 mm, vias 2 -> 0
- net /VGH: track 26.5 -> 0.00 mm, vias 2 -> 0
- net UPDI: track 25.7 -> 0.00 mm, vias 1 -> 0
- net DISP_BUSY: track 25.2 -> 0.00 mm, vias 2 -> 0
- net DISP_DC: track 25.0 -> 0.00 mm, vias 2 -> 0
- net DISP_RES#: track 20.5 -> 0.00 mm
- net EXTCOMIN: track 0.00 -> 20.1 mm, vias 0 -> 2
- net VBAT_OK: track 0.00 -> 19.1 mm, vias 0 -> 2
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- added copper zone on F.Cu, net /LBOOST
Other:
- board size 80 x 32 mm -> 80 x 30 mm
